File: pcb/module S-RX28_rev3.3 644.brd (EAGLE design)
At the start: 44.5 x 30.5 mm, 47 parts, among them U1 ATMEGA644PA-AU, Y2 16MHz

Commit message: added docs
Parts:
- C1, C4: value 0.1uF -> 100nF
- C3: value 0.1uf -> 100nF
Connections:
- net CH2 renamed CH2/RXD0
- net CH3 renamed CH3/TXD0
