File: pcb/module S-RX28_rev3.3 644.sch (EAGLE design)
At the start: 46 parts, among them U1 ATMEGA644PA-AU, Y2 16MHz

Commit message: added docs
Parts:
- C1, C4: value 0.1uF -> 100nF
- C3: value 0.1uf -> 100nF
Connections:
- net CH2 renamed CH2/RXD0
- net CH3 renamed CH3/TXD0
Other:
- note added: "Created by Albert Kravcov"
- note removed: "Warum?"
- moved on the sheet: -, 10K, 1K, 470, 5V, A60, A65, ANT, B+, B-, BX, C2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
