File: pcb/module S-RX28_rev05 644.brd (EAGLE design)
At the start: 44.5 x 30.5 mm, 47 parts, among them U1 ATMEGA644PA-AU, Y2 16MHz

Commit message: new PCB revision
Parts:
- added BUZZ: JUMPER-SMT_2_NC_PASTE_SILK, SparkFun-Jumpers:SMT-JUMPER_2_NC_PASTE_SILK
- added D2: (no value), SparkFun-LED:LED-0603
- added R9: 330, SparkFun-Resistors:0603
- moved R8 12.5 mm to (26.7, 14.0), turned to 0 degrees
- moved C5 9.67 mm to (8.89, 26.7), turned to 270 degrees
- moved R2 3.81 mm to (24.1, 27.9)
- moved R3 3.81 mm to (27.9, 27.9)
- moved RSSI 3.54 mm to (-1.27, 17.0)
- moved R4 2.67 mm to (0.00, 20.4)
- moved GOOGLE_IO 1.27 mm to (38.1, 6.35)
- moved D1 1.27 mm to (0.00, 18.5)
- moved S2 1.14 mm to (32.8, 19.4)
- moved GND•5V•SCL•SDA 0.72 mm to (12.7, 30.5)
- moved B+ 0.51 mm to (5.08, 23.9)
- moved C4 0.51 mm to (5.08, 7.62)
- moved B- 0.51 mm to (5.08, 27.2)
- renumbered Y2 to Y1
Connections:
- new net N$2: B+.TP, BUZZ.1
- new net RED1: D2.A, R9.2
- net 5V: now also R9.1
- net BUZZER: now also BUZZ.2; no longer B+.TP
- net GND: now also D2.C
- net RES: now also U1.40
Routing:
- net N$2: track 0.00 -> 9.61 mm, vias 0 -> 1
- net BUZZER: track 22.0 -> 29.2 mm, vias 0 -> 3
- net RES: track 64.3 -> 71.2 mm, vias 1 -> 3
- net 5V: track 130.0 -> 135.8 mm
- net VIDEO: track 29.0 -> 23.4 mm
- net RSSI_IN: track 31.9 -> 36.0 mm
- net C2: track 7.30 -> 3.44 mm
- net C1: track 9.94 -> 6.10 mm
- net N$4: track 6.14 -> 9.93 mm
- net N$3: track 9.68 -> 13.5 mm
- net BT0: track 26.2 -> 22.5 mm
- net LED: track 15.5 -> 18.4 mm
- net RED1: track 0.00 -> 1.88 mm
- net CH1: track 27.8 -> 29.7 mm
- net A_L: track 14.7 -> 13.4 mm
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Other:
- board text added: "644PA-AU"
- board text added: "MODULE"
- board text added: "OSD"
- board text added: "PWR"
- board text added: "• GND | GND | 5V | TX | RX | DTR"
- board text removed: "644PA-AU 1284P-AU"
- board text removed: "G•G•5V•TX•RX•DTR"
