File: pcb/module S-RX28_rev05 644.sch (EAGLE design)
At the start: 46 parts, among them U1 ATMEGA644PA-AU, Y2 16MHz

Commit message: new PCB revision
Parts:
- added BUZZ: JUMPER-SMT_2_NC_PASTE_SILK, SparkFun-Jumpers:JUMPER-SMT_2_NC_PASTE_SILK
- added D2: (no value), SparkFun-LED:LED0603
- added R9: 330, SparkFun-Resistors:0.05OHM-0603-1/5W-1%
- renumbered Y2 to Y1
Connections:
- new net N$2: B+.TP, BUZZ.1
- new net RED1: D2.A, R9.2
- net 5V: now also R9.1
- net BUZZER: now also BUZZ.2; no longer B+.TP
- net GND: now also D2.C
- net RES: now also U1.PB0
Other:
- moved on the sheet: C2
Changed lines of the file:
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@@
 <part name="GND5" library="supply1" library_urn="urn:adsk.eagle:library:371" deviceset="GND" device=""/>
 <part name="R5" library="SparkFun-Resistors" library_urn="urn:adsk.eagle:library:532" deviceset="0.05OHM" device="-0603-1/5W-1%" package3d_urn="urn:adsk.eagle:package:39650/1" value="1k"/>
-<part name="Y2" library="SparkFun-Clocks" library_urn="urn:adsk.eagle:library:511" deviceset="RESONATOR-16MHZ" device="SMD_3.2X1.3" package3d_urn="urn:adsk.eagle:package:37551/1" value="16MHz"/>
+<part name="Y1" library="SparkFun-Clocks" library_urn="urn:adsk.eagle:library:511" deviceset="RESONATOR-16MHZ" device="SMD_3.2X1.3" package3d_urn="urn:adsk.eagle:package:37551/1" value="16MHz"/>
 <part name="1K" library="SparkFun-Resistors" library_urn="urn:adsk.eagle:library:532" deviceset="0.27OHM" device="-0603-1/10W-1%" package3d_urn="urn:adsk.eagle:package:39650/1" value=""/>
 <part name="470" library="SparkFun-Resistors" library_urn="urn:adsk.eagle:library:532" deviceset="0.27OHM" device="-0603-1/10W-1%" package3d_urn="urn:adsk.eagle:package:39650/1" value=""/>
@@
 <part name="U1" library="ATMEGA644PA-AU" deviceset="ATMEGA644PA-AU" device=""/>
 <part name="GND13" library="supply1" library_urn="urn:adsk.eagle:library:371" deviceset="GND" device=""/>
+<part name="D2" library="SparkFun-LED" library_urn="urn:adsk.eagle:library:529" deviceset="LED" device="0603" package3d_urn="urn:adsk.eagle:package:39354/1"/>
+<part name="R9" library="SparkFun-Resistors" library_urn="urn:adsk.eagle:library:532" deviceset="0.05OHM" device="-0603-1/5W-1%" package3d_urn="urn:adsk.eagle:package:39650/1" value="330"/>
+<part name="GND10" library="supply1" library_urn="urn:adsk.eagle:library:371" deviceset="GND" device=""/>
+<part name="BUZZ" library="SparkFun-Jumpers" library_urn="urn:adsk.eagle:library:528" deviceset="JUMPER-SMT_2_NC_PASTE" device="_SILK" package3d_urn="urn:adsk.eagle:package:39282/1"/>
 </parts>
 <sheets>
@@
 <attribute name="VALUE" x="116.84" y="11.684" size="1.778" layer="96" font="vector" rot="R180" align="top-center"/>
 </instance>
-<instance part="Y2" gate="G$1" x="35.56" y="121.92" smashed="yes" rot="R270">
+<instance part="Y1" gate="G$1" x="35.56" y="121.92" smashed="yes" rot="R270">
 <attribute name="NAME" x="33.02" y="120.142" size="1.778" layer="95" font="vector" rot="R270" align="center-right"/>
 <attribute name="VALUE" x="37.592" y="121.92" size="1.778" layer="96" font="vector" rot="R270" align="bottom-center"/>
@@
 <attribute name="VALUE" x="123.444" y="68.58" size="1.778" layer="96" font="vector" rot="R90" align="top-center"/>
 </instance>
-<instance part="C2" gate="G$1" x="88.9" y="137.16" smashed="yes">
-<attribute name="NAME" x="89.916" y="137.795" size="1.778" layer="95"/>
-<attribute name="VALUE" x="89.916" y="132.969" size="1.778" layer="96"/>
-</instance>
-<instance part="P+8" gate="G$1" x="88.9" y="142.24" smashed="yes">
-<attribute name="VALUE" x="87.884" y="145.796" size="1.778" layer="96"/>
-</instance>
-<instance part="GND16" gate="1" x="88.9" y="116.84" smashed="yes">
-<attribute name="VALUE" x="86.36" y="114.3" size="1.778" layer="96"/>
+<instance part="C2" gate="G$1" x="83.82" y="137.16" smashed="yes">
+<attribute name="NAME" x="84.836" y="137.795" size="1.778" layer="95"/>
+<attribute name="VALUE" x="84.836" y="132.969" size="1.778" layer="96"/>
+</instance>
+<instance part="P+8" gate="G$1" x="83.82" y="142.24" smashed="yes">
+<attribute name="VALUE" x="82.804" y="145.796" size="1.778" layer="96"/>
+</instance>
+<instance part="GND16" gate="1" x="83.82" y="116.84" smashed="yes">
+<attribute name="VALUE" x="81.28" y="114.3" size="1.778" layer="96"/>
 </instance>
 <instance part="R6" gate="G$1" x="195.58" y="137.16" smashed="yes">
@@
 <instance part="GND13" gate="1" x="12.7" y="7.62" smashed="yes">
 <attribute name="VALUE" x="10.16" y="5.08" size="1.778" layer="96"/>
+</instance>
+<instance part="D2" gate="G$1" x="99.06" y="127" smashed="yes">
+<attribute name="NAME" x="95.631" y="122.428" size="1.778" layer="95" font="vector" rot="R90"/>
+<attribute name="VALUE" x="100.965" y="122.428" size="1.778" layer="96" font="vector" rot="R90" align="top-left"/>
+</instance>
+<instance part="R9" gate="G$1" x="99.06" y="134.62" smashed="yes" rot="R270">
+<attribute name="NAME" x="100.584" y="134.62" size="1.778" layer="95" font="vector" rot="R270" align="bottom-center"/>
+<attribute name="VALUE" x="97.536" y="134.62" size="1.778" layer="96" font="vector" rot="R270" align="top-center"/>
+</instance>
+<instance part="GND10" gate="1" x="99.06" y="116.84" smashed="yes">
+<attribute name="VALUE" x="96.52" y="114.3" size="1.778" layer="96"/>
+</instance>
+<instance part="BUZZ" gate="G$1" x="142.24" y="83.82" smashed="yes" rot="R90">
+<attribute name="NAME" x="139.7" y="81.28" size="1.778" layer="95" font="vector" rot="R90"/>
+<attribute name="VALUE" x="144.78" y="81.28" size="1.778" layer="96" font="vector" rot="R90" align="top-left"/>
 </instance>
 </instances>
@@
 <wire x1="27.94" y1="121.92" x2="25.4" y2="121.92" width="0.1524" layer="91"/>
 <pinref part="GND8" gate="1" pin="GND"/>
-<pinref part="Y2" gate="G$1" pin="2"/>
+<pinref part="Y1" gate="G$1" pin="2"/>
 </segment>
 <segment>
@@
 <pinref part="C2" gate="G$1" pin="-"/>
 <pinref part="GND16" gate="1" pin="GND"/>
-<wire x1="88.9" y1="119.38" x2="88.9" y2="132.08" width="0.1524" layer="91"/>
+<wire x1="83.82" y1="119.38" x2="83.82" y2="132.08" width="0.1524" layer="91"/>
 </segment>
 <segment>
@@
 <pinref part="C5" gate="G$1" pin="2"/>
 </segment>
+<segment>
+<pinref part="D2" gate="G$1" pin="C"/>
+<pinref part="GND10" gate="1" pin="GND"/>
+<wire x1="99.06" y1="121.92" x2="99.06" y2="119.38" width="0.1524" layer="91"/>
+</segment>
 </net>
 <net name="RED" class="0">
@@
 <pinref part="P+8" gate="G$1" pin="3.3V"/>
 <pinref part="C2" gate="G$1" pin="+"/>
-<wire x1="88.9" y1="142.24" x2="88.9" y2="139.7" width="0.1524" layer="91"/>
+<wire x1="83.82" y1="142.24" x2="83.82" y2="139.7" width="0.1524" layer="91"/>
 </segment>
 <segment>
@@
 <pinref part="C5" gate="G$1" pin="1"/>
 </segment>
+<segment>
+<pinref part="R9" gate="G$1" pin="1"/>
+<wire x1="99.06" y1="144.78" x2="99.06" y2="139.7" width="0.1524" layer="91"/>
+<label x="99.06" y="144.78" size="1.778" layer="95" rot="R90" xref="yes"/>
+</segment>
 </net>
 <net name="VIDEO" class="1">
@@
 <label x="187.96" y="91.44" size="1.778" layer="95" xref="yes"/>
 </segment>
+<segment>
+<pinref part="U1" gate="A" pin="PB0"/>
+<wire x1="17.78" y1="50.8" x2="12.7" y2="50.8" width="0.1524" layer="91"/>
+<label x="12.7" y="50.8" size="1.778" layer="95" rot="R180" xref="yes"/>
+</segment>
 </net>
 <net name="DTR" class="0">
@@
 </segment>
 <segment>
-<pinref part="Y2" gate="G$1" pin="1"/>
+<pinref part="Y1" gate="G$1" pin="1"/>
 <wire x1="35.56" y1="124.46" x2="45.72" y2="124.46" width="0.1524" layer="91"/>
 <label x="45.72" y="124.46" size="1.778" layer="95" xref="yes"/>
@@
 </segment>
 <segment>
-<pinref part="Y2" gate="G$1" pin="3"/>
+<pinref part="Y1" gate="G$1" pin="3"/>
 <wire x1="35.56" y1="119.38" x2="45.72" y2="119.38" width="0.1524" layer="91"/>
 <label x="45.72" y="119.38" size="1.778" layer="95" xref="yes"/>
@@
 </segment>
 <segment>
-<wire x1="142.24" y1="76.2" x2="142.24" y2="83.82" width="0.1524" layer="91"/>
-<label x="142.24" y="83.82" size="1.778" layer="95" rot="R90" xref="yes"/>
-<pinref part="B+" gate="G$1" pin="TP"/>
+<pinref part="BUZZ" gate="G$1" pin="2"/>
+<wire x1="142.24" y1="88.9" x2="142.24" y2="93.98" width="0.1524" layer="91"/>
+<label x="142.24" y="93.98" size="1.778" layer="95" rot="R90" xref="yes"/>
 </segment>
 </net>
@@
 </segment>
 </net>
+<net name="RED1" class="0">
+<segment>
+<pinref part="D2" gate="G$1" pin="A"/>
+<pinref part="R9" gate="G$1" pin="2"/>
+</segment>
+</net>
+<net name="N$2" class="0">
+<segment>
+<pinref part="BUZZ" gate="G$1" pin="1"/>
+<pinref part="B+" gate="G$1" pin="TP"/>
+<wire x1="142.24" y1="78.74" x2="142.24" y2="76.2" width="0.1524" layer="91"/>
+</segment>
+</net>
