File: pcb/module S-RX28_rev06 644.brd (EAGLE design)
At the start: 44.5 x 30.5 mm, 51 parts, among them U1 ATMEGA644PA-AU, Y1 16MHz

Commit message: OSD Finder Mode + New PCB revision (with mounting hole)
Parts:
- added U$3, U$4, U$5: FIDUCIALUFIDUCIAL, SparkFun-Aesthetics:FIDUCIAL-MICRO
- renumbered B+ to BZ+, B- to BZ-, JUMPER1 to JUMP1
Routing:
- net RES: track 77.9 -> 65.9 mm, vias 1 -> 3
Other:
- outline, holes or cut-outs redrawn
- board text added: "U1"
- board text removed: "644PA-AU"

Commit message: cleanup
Parts:
- R6: value 10R -> 0R
Changed lines of the file:
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@@
 <attribute name="VALUE" x="29.21" y="7.62" size="0.4064" layer="27"/>
 </element>
-<element name="R6" library="resistor" library_urn="urn:adsk.eagle:library:348" package="R0603" package3d_urn="urn:adsk.eagle:package:23555/2" value="10R" x="22.987" y="8.89" smashed="yes" rot="R90">
+<element name="R6" library="resistor" library_urn="urn:adsk.eagle:library:348" package="R0603" package3d_urn="urn:adsk.eagle:package:23555/2" value="0R" x="22.987" y="8.89" smashed="yes" rot="R90">
 <attribute name="NAME" x="24.511" y="8.255" size="0.7112" layer="25" font="vector" ratio="20" rot="R90"/>
 <attribute name="VALUE" x="25.527" y="8.255" size="1.27" layer="27" rot="R90"/>
