File: pcb/module S-RX28_rev06 644.sch (EAGLE design)
At the start: 50 parts, among them U1 ATMEGA644PA-AU, Y1 16MHz

Commit message: OSD Finder Mode + New PCB revision (with mounting hole)
Parts:
- added U$3, U$4, U$5: FIDUCIALUFIDUCIAL, SparkFun-Aesthetics:FIDUCIALUFIDUCIAL
- renumbered B+ to BZ+, B- to BZ-, FLASHING to JUMP1
Changed lines of the file:
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@@
 <part name="S2" library="SparkFun-Switches" library_urn="urn:adsk.eagle:library:535" deviceset="JOYSTICK_MINI" device="" package3d_urn="urn:adsk.eagle:package:40157/1"/>
 <part name="GND2" library="supply1" library_urn="urn:adsk.eagle:library:371" deviceset="GND" device=""/>
-<part name="B+" library="testpad" library_urn="urn:adsk.eagle:library:385" deviceset="TP" device="TP17SQ" package3d_urn="urn:adsk.eagle:package:27977/1"/>
-<part name="B-" library="testpad" library_urn="urn:adsk.eagle:library:385" deviceset="TP" device="TP17SQ" package3d_urn="urn:adsk.eagle:package:27977/1"/>
+<part name="BZ+" library="testpad" library_urn="urn:adsk.eagle:library:385" deviceset="TP" device="TP17SQ" package3d_urn="urn:adsk.eagle:package:27977/1"/>
+<part name="BZ-" library="testpad" library_urn="urn:adsk.eagle:library:385" deviceset="TP" device="TP17SQ" package3d_urn="urn:adsk.eagle:package:27977/1"/>
 <part name="GND6" library="supply1" library_urn="urn:adsk.eagle:library:371" deviceset="GND" device=""/>
 <part name="SCK" library="testpad" library_urn="urn:adsk.eagle:library:385" deviceset="TPSQ" device="B1,27" package3d_urn="urn:adsk.eagle:package:27944/2" value="TPSQB1,27"/>
@@
 <part name="GND10" library="supply1" library_urn="urn:adsk.eagle:library:371" deviceset="GND" device=""/>
 <part name="BUZZ" library="SparkFun-Jumpers" library_urn="urn:adsk.eagle:library:528" deviceset="JUMPER-SMT_2_NC_PASTE" device="_SILK" package3d_urn="urn:adsk.eagle:package:39282/1"/>
-<part name="FLASHING" library="SparkFun-Jumpers" library_urn="urn:adsk.eagle:library:528" deviceset="JUMPER-SMT_2_NC_PASTE" device="_SILK" package3d_urn="urn:adsk.eagle:package:39282/1"/>
+<part name="JUMP1" library="SparkFun-Jumpers" library_urn="urn:adsk.eagle:library:528" deviceset="JUMPER-SMT_2_NC_PASTE" device="_SILK" package3d_urn="urn:adsk.eagle:package:39282/1"/>
+<part name="U$3" library="SparkFun-Aesthetics" library_urn="urn:adsk.eagle:library:507" deviceset="FIDUCIAL" device="UFIDUCIAL" package3d_urn="urn:adsk.eagle:package:37111/1"/>
+<part name="U$4" library="SparkFun-Aesthetics" library_urn="urn:adsk.eagle:library:507" deviceset="FIDUCIAL" device="UFIDUCIAL" package3d_urn="urn:adsk.eagle:package:37111/1"/>
+<part name="U$5" library="SparkFun-Aesthetics" library_urn="urn:adsk.eagle:library:507" deviceset="FIDUCIAL" device="UFIDUCIAL" package3d_urn="urn:adsk.eagle:package:37111/1"/>
 </parts>
 <sheets>
@@
 <attribute name="VALUE" x="93.98" y="-35.56" size="1.778" layer="96"/>
 </instance>
-<instance part="B+" gate="G$1" x="142.24" y="73.66" smashed="yes" rot="R180">
+<instance part="BZ+" gate="G$1" x="142.24" y="73.66" smashed="yes" rot="R180">
 <attribute name="NAME" x="143.51" y="72.39" size="1.778" layer="95" rot="R180"/>
 <attribute name="TP_SIGNAL_NAME" x="140.97" y="74.93" size="1.778" layer="97" rot="R180"/>
 </instance>
-<instance part="B-" gate="G$1" x="142.24" y="63.5" smashed="yes">
+<instance part="BZ-" gate="G$1" x="142.24" y="63.5" smashed="yes">
 <attribute name="NAME" x="140.97" y="64.77" size="1.778" layer="95"/>
 <attribute name="TP_SIGNAL_NAME" x="143.51" y="62.23" size="1.778" layer="97"/>
@@
 <instance part="BUZZ" gate="G$1" x="142.24" y="83.82" smashed="yes" rot="R90">
 <attribute name="NAME" x="139.7" y="81.28" size="1.778" layer="95" font="vector" rot="R90"/>
-<attribute name="VALUE" x="144.78" y="81.28" size="1.778" layer="96" font="vector" rot="R90" align="top-left"/>
-</instance>
-<instance part="FLASHING" gate="G$1" x="154.94" y="83.82" smashed="yes" rot="R90">
+</instance>
+<instance part="JUMP1" gate="G$1" x="154.94" y="83.82" smashed="yes" rot="R90">
 <attribute name="NAME" x="152.4" y="81.28" size="1.778" layer="95" font="vector" rot="R90"/>
-<attribute name="VALUE" x="157.48" y="81.28" size="1.778" layer="96" font="vector" rot="R90" align="top-left"/>
-</instance>
+</instance>
+<instance part="U$3" gate="G$1" x="-20.32" y="-10.16" smashed="yes"/>
+<instance part="U$4" gate="G$1" x="-20.32" y="-15.24" smashed="yes"/>
+<instance part="U$5" gate="G$1" x="-20.32" y="-20.32" smashed="yes"/>
 </instances>
 <busses>
@@
 </segment>
 <segment>
-<pinref part="B-" gate="G$1" pin="TP"/>
+<pinref part="BZ-" gate="G$1" pin="TP"/>
 <wire x1="142.24" y1="60.96" x2="142.24" y2="55.88" width="0.1524" layer="91"/>
 <pinref part="GND6" gate="1" pin="GND"/>
@@
 </segment>
 <segment>
-<pinref part="FLASHING" gate="G$1" pin="1"/>
+<pinref part="JUMP1" gate="G$1" pin="1"/>
 <wire x1="154.94" y1="78.74" x2="154.94" y2="73.66" width="0.1524" layer="91"/>
 <label x="154.94" y="73.66" size="1.778" layer="95" rot="R270" xref="yes"/>
@@
 <segment>
 <pinref part="BUZZ" gate="G$1" pin="1"/>
-<pinref part="B+" gate="G$1" pin="TP"/>
+<pinref part="BZ+" gate="G$1" pin="TP"/>
 <wire x1="142.24" y1="78.74" x2="142.24" y2="76.2" width="0.1524" layer="91"/>
 </segment>
@@
 </segment>
 <segment>
-<pinref part="FLASHING" gate="G$1" pin="2"/>
+<pinref part="JUMP1" gate="G$1" pin="2"/>
 <wire x1="154.94" y1="88.9" x2="154.94" y2="93.98" width="0.1524" layer="91"/>
 <label x="154.94" y="93.98" size="1.778" layer="95" rot="R90" xref="yes"/>

Commit message: cleanup
Parts:
- R6: value 10R -> 0R
Changed lines of the file:
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@@
 <part name="P+8" library="SparkFun" deviceset="3.3V" device="" value="VCC"/>
 <part name="GND16" library="supply1" deviceset="GND" device=""/>
-<part name="R6" library="resistor" library_urn="urn:adsk.eagle:library:348" deviceset="R-EU_" device="R0603" package3d_urn="urn:adsk.eagle:package:23555/2" value="10R"/>
+<part name="R6" library="resistor" library_urn="urn:adsk.eagle:library:348" deviceset="R-EU_" device="R0603" package3d_urn="urn:adsk.eagle:package:23555/2" value="0R"/>
 <part name="GND7" library="supply1" deviceset="GND" device=""/>
 <part name="P+2" library="SparkFun" deviceset="3.3V" device="" value="VCC"/>
