File: pcb/adapter RX2189.brd (EAGLE design)
At the start: 39.4 x 30.5 mm, 26 parts

Commit message: documentation update
Parts:
- added C1: (no value), resistor:C1206K
- added C2: 470uf, SparkFun-Passives:EIA7343
- added L1: (no value), rcl:POWER-CHOKE_WE-TPC
- added L2: NR4018T101M, NRS5020T220MMGJ:INDM4949X200N
- added R1, R2, R3: (no value), resistor:R0603
- moved 1 1.02 mm to (26.9, 13.2)
- moved 10 1.02 mm to (26.9, 31.5)
- moved 2 1.02 mm to (26.9, 15.2)
- moved 3 1.02 mm to (26.9, 17.3)
- moved 4 1.02 mm to (26.9, 19.3)
- moved 5 1.02 mm to (26.9, 21.3)
- moved 6 1.02 mm to (26.9, 23.4)
- moved 7 1.02 mm to (26.9, 25.4)
- moved 8 1.02 mm to (26.9, 27.4)
- moved 9 1.02 mm to (26.9, 29.5)
- moved 11 1.02 mm to (4.06, 31.5)
- moved 12 1.02 mm to (4.06, 29.5)
- moved 13 1.02 mm to (4.06, 27.4)
- moved J1 1.02 mm to (35.3, 31.8)
- moved J2 1.02 mm to (35.3, 29.2)
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Connections:
- new net 5VFILTERED: 8.TP, 9.TP, C1.1, L2.2
- new net N$1: 2.TP, C2.A
- net 5V: now also L2.1, R1.2, R2.2, R3.2; no longer 8.TP
- net BX: no longer 9.TP
- net CH1: now also 5.TP, R3.1
- net CH2: now also R2.1
- net CH3: now also R1.1; no longer 5.TP
- net GND: now also C1.2
- net VID: now also C2.C; no longer 2.TP
Routing:
- net GND: track 19.6 -> 59.2 mm, vias 2 -> 4
- net 5VFILTERED: track 0.00 -> 30.5 mm, vias 0 -> 3
- net CH1: track 0.00 -> 15.1 mm, vias 0 -> 1
- net CH2: track 7.73 -> 15.5 mm, vias 0 -> 1
- net BX: track 7.28 -> 0.00 mm
- net A65: track 7.71 -> 13.3 mm, vias 0 -> 1
- net N$1: track 0.00 -> 4.71 mm
- net CH3: track 18.6 -> 14.6 mm, vias 1 -> 0
- net ANT: track 4.96 -> 7.60 mm
- net 5V: track 17.0 -> 14.4 mm
- net VID: track 7.92 -> 5.76 mm
- added copper zone on layer 16, net GND
Other:
- outline, holes or cut-outs redrawn
- board text added: "REV 0.2"
- board text removed: "REV 0.1"
