File: pcb/adapter RX2189.sch (EAGLE design)
At the start: 25 parts

Commit message: documentation update
Parts:
- added C1: (no value), resistor:C-EUC1206K
- added C2: 470uf, SparkFun-Passives:CAP_POL7343
- added L1: (no value), rcl:L-EUWE-TPC
- added L2: NR4018T101M, NRS5020T220MMGJ:NRS5020T220MMGJ
- added R1, R2, R3: (no value), resistor:R-EU_R0603
Connections:
- new net 5VFILTERED: 8.TP, 9.TP, C1.1, L2.2
- new net N$1: 2.TP, C2.+
- net 5V: now also L2.1, R1.2, R2.2, R3.2; no longer 8.TP
- net BX: no longer 9.TP
- net CH1: now also 5.TP, R3.1
- net CH2: now also R2.1
- net CH3: now also R1.1; no longer 5.TP
- net GND: now also C1.2
- net VID: now also C2.-; no longer 2.TP
